Commit message: update material.xacro and mobile_diff_robot.xacro

File: diff_description/urdf/material.xacro (robot description, xacro)
@@ -7,3 +7,12 @@
         <color rgba="0.0 0.0 0.0 1.0" />
     </material>
+    <material name="grey">
+        <color rgba="0.5 0.5 0.5 1" />
+    </material>
+    <material name="orange">
+        <color rgba="1.0 0.5 0 1" />
+    </material>
+    <material name="yellow">
+        <color rgba="1.0 1.0 0 1" />
+    </material>
 </robot>

File: diff_description/urdf/mobile_diff_robot.xacro (robot description, xacro)
@@ -4,3 +4,6 @@
     <xacro:include filename="inertial.xacro" />
     <xacro:include filename="mobile_base.xacro" />
+    <xacro:include filename="mobile_base_gazebo.xacro" />
+    <xacro:include filename="camera.xacro" />
+    <xacro:include filename="lidar.xacro" />
 </robot>
